File: Bridge universal/kicad/toshibridge.sch (KiCad schematic (older format))
At the start: 27 parts

Commit message: Añadimos un conector de 2 pines en el esquemático del bridge universal.
Parts:
- added P?: CONN_2, symbol CONN_2
Connections:
- net RX_1: now also P?.1 (P1)
- net TX_1: now also P?.2 (PM)
- net T1: no longer names the net of IC?.6 (PB2)
Changed lines of the file:
@@
-EESchema Schematic File Version 2  date Mon 25 Apr 2011 13:48:49 ART
+EESchema Schematic File Version 2  date Wed 27 Apr 2011 02:07:39 ART
 LIBS:power
 LIBS:ATXMEGA-A4-QFN
@@
 Sheet 1 1
 Title ""
-Date "25 apr 2011"
+Date "27 apr 2011"
 Rev ""
 Comp ""
@@
 Comment4 ""
 $EndDescr
+Text Label 7850 6500 2    60   ~ 0
+TX_1
+Text Label 7850 6300 2    60   ~ 0
+RX_1
+$Comp
+L CONN_2 P?
+U 1 1 4DB7A406
+P 8200 6400
+F 0 "P?" V 8150 6400 40  0000 C CNN
+F 1 "CONN_2" V 8250 6400 40  0000 C CNN
+	1    8200 6400
+	1    0    0    -1
+$EndComp
 Connection ~ 7850 5700
 Wire Wire Line
@@
 Text Label 9600 4250 0    60   ~ 0
 DCLK_TOSHI
-Text Label 7000 3850 2    60   ~ 0
-T1
 Text Label 8200 4850 3    60   ~ 0
 RX_1

Commit message: Se sustituyeron todos los footprint 0805 a 1206, se agrando la placa en consecuencia y se eliminaron las pistas debajo de la camara.
Parts:
- C4: renamed from C?; value C -> 100nF
- R1, R2: renamed from R?; value R -> 270
- gave numbers to parts that had none: 25

Commit message: Se cambia el footprint del oscilador, se colocan las vias para cables, no para placa bifaz.
Parts:
- added R? (x2): 270, symbol R
Connections:
- net +3.3V: now also R?.2, R?.2; no longer D3.1 (A), D4.1 (A)
- new net: D3.1 (A), R?.1
- new net: D4.1 (A), R?.1
Other:
- moved on the sheet: P4
